File: hover_cello/pcb_layouts/hover_controller_v3/hover_controller_v3.brd (EAGLE design)
At the start: 101.6 x 44.5 mm, 33 parts, among them IC1 74LS279N, U1 L298

Commit message: almost finished routing PCB
Routing:
- net CTRL_1: track 17.8 -> 107.9 mm, vias 0 -> 2
- net CTRL_2: track 15.7 -> 105.5 mm, vias 0 -> 2
- net CTRL_3: track 18.2 -> 98.8 mm, vias 0 -> 1
- net VCC: track 96.1 -> 169.5 mm
- net N$4: track 0.00 -> 65.9 mm, vias 0 -> 1
- net N$18: track 42.9 -> 108.4 mm, vias 0 -> 1
- net CTRL_4: track 15.7 -> 77.0 mm
- net N$2: track 0.00 -> 59.9 mm
- net CTRL_5: track 17.5 -> 69.3 mm, vias 0 -> 1
- net S1: track 5.08 -> 48.7 mm
- net N$1: track 0.00 -> 29.3 mm
- net N$3: track 0.00 -> 28.3 mm
- net S3: track 5.08 -> 22.8 mm
- net R4: track 13.8 -> 29.0 mm
- net N$15: track 0.00 -> 13.4 mm
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